Commit message: xacro directory bugfix

File: ros2_ws_head/src/head_bringup/urdf/tele.urdf.xacro (robot description, xacro)
@@ -35,20 +35,20 @@
     <visual>
       <origin xyz="0 0 0" rpy="0 0 1.57"/>
-      <geometry><mesh filename="package://easy_way/meshes/lower_bottom.stl" scale="0.001 0.001 0.001"/></geometry>
+      <geometry><mesh filename="package://head_bringup/meshes/lower_bottom.stl" scale="0.001 0.001 0.001"/></geometry>
       <material name="tele_grey"><color rgba="0.7 0.7 0.7 1"/></material>
     </visual>
     <visual>
       <origin xyz="0 0 0" rpy="0 0 1.57"/>
-      <geometry><mesh filename="package://easy_way/meshes/upper_bottom.stl" scale="0.001 0.001 0.001"/></geometry>
+      <geometry><mesh filename="package://head_bringup/meshes/upper_bottom.stl" scale="0.001 0.001 0.001"/></geometry>
       <material name="tele_grey"/>
     </visual>
     <visual>
       <origin xyz="0 0 0" rpy="0 0 1.57"/>
-      <geometry><mesh filename="package://easy_way/meshes/mid_section.stl" scale="0.001 0.001 0.001"/></geometry>
+      <geometry><mesh filename="package://head_bringup/meshes/mid_section.stl" scale="0.001 0.001 0.001"/></geometry>
       <material name="tele_grey"/>
     </visual>
     <visual>
       <origin xyz="0 0 0" rpy="0 0 1.57"/>
-      <geometry><mesh filename="package://easy_way/meshes/chest.stl" scale="0.001 0.001 0.001"/></geometry>
+      <geometry><mesh filename="package://head_bringup/meshes/chest.stl" scale="0.001 0.001 0.001"/></geometry>
       <material name="tele_grey"/>
     </visual>
@@ -64,5 +64,5 @@
     <visual>
       <origin xyz="-0.02 0 0" rpy="0 0 1.57"/>
-      <geometry><mesh filename="package://easy_way/meshes/head_body_joint.stl" scale="0.001 0.001 0.001"/></geometry>
+      <geometry><mesh filename="package://head_bringup/meshes/head_body_joint.stl" scale="0.001 0.001 0.001"/></geometry>
       <material name="tele_blue"><color rgba="0 0 0.8 1"/></material>
     </visual>
@@ -83,5 +83,5 @@
     <visual>
       <origin xyz="0 0 0" rpy="0 0 1.57"/>
-      <geometry><mesh filename="package://easy_way/meshes/head.stl" scale="0.001 0.001 0.001"/></geometry>
+      <geometry><mesh filename="package://head_bringup/meshes/head.stl" scale="0.001 0.001 0.001"/></geometry>
       <material name="tele_grey"/>
     </visual>

Commit message: urdf tilt axis reversed

File: ros2_ws_head/src/head_bringup/urdf/tele.urdf.xacro (robot description, xacro)
@@ -77,5 +77,5 @@
     <child link="tele_head_link"/>
     <origin xyz="0 0 ${tilt_joint_z}" rpy="0 0 0"/>
-    <axis xyz="0 1 0"/>
+    <axis xyz="0 -1 0"/>
     <limit lower="-1.57" upper="1.57" effort="10" velocity="1.0"/>
   </joint>
